Commit message: updated the skeleton urdf

File: urdf/asbr.urdf (robot description, URDF)
Before this commit: robot ur5e_robot, 35 links, 34 joints
Links:
- added link camera_link
Joints:
- added joint camera_joint: type fixed, parent tool0, child camera_link, origin xyz=-0.15 -0.05 0.015 rpy=0 0 0, axis 0 0 1

Commit message: generated the main urdf using xacro

File: urdf/asbr.urdf (robot description, URDF)
Before this commit: robot ur5e_robot, 36 links, 35 joints
Joints:
- joint robotiq_85_base_joint: parent ur_to_robotiq_link -> gripper_mount_link

Commit message: update the main.xacro and launch files

File: urdf/asbr.urdf (robot description, URDF)
Before this commit: robot ur5e_robot, 36 links, 35 joints
Links:
- removed link gripper_mount_link
- removed link robotiq_85_base_link
- removed link robotiq_85_left_finger_link
- removed link robotiq_85_left_finger_tip_link
- removed link robotiq_85_left_inner_knuckle_link
- removed link robotiq_85_left_knuckle_link
- removed link robotiq_85_right_finger_link
- removed link robotiq_85_right_finger_tip_link
- removed link robotiq_85_right_inner_knuckle_link
- removed link robotiq_85_right_knuckle_link
- removed link ur_to_robotiq_link
- link base_link_inertia: geometry collision mesh filename=package://ur_description/meshes/ur5/collision/base.stl; visual mesh filename=package://ur_description/meshes/ur5/visual/base.dae
- link forearm_link: geometry collision mesh filename=package://ur_description/meshes/ur5/collision/forearm.stl; visual mesh filename=package://ur_description/meshes/ur5/visual/forearm.dae
- link shoulder_link: geometry collision mesh filename=package://ur_description/meshes/ur5/collision/shoulder.stl; visual mesh filename=package://ur_description/meshes/ur5/visual/shoulder.dae
- link upper_arm_link: geometry collision mesh filename=package://ur_description/meshes/ur5/collision/upperarm.stl; visual mesh filename=package://ur_description/meshes/ur5/visual/upperarm.dae
- link wrist_1_link: geometry collision mesh filename=package://ur_description/meshes/ur5/collision/wrist1.stl; visual mesh filename=package://ur_description/meshes/ur5/visual/wrist1.dae
- link wrist_2_link: geometry collision mesh filename=package://ur_description/meshes/ur5/collision/wrist2.stl; visual mesh filename=package://ur_description/meshes/ur5/visual/wrist2.dae
- link wrist_3_link: geometry collision mesh filename=package://ur_description/meshes/ur5/collision/wrist3.stl; visual mesh filename=package://ur_description/meshes/ur5/visual/wrist3.dae
Joints:
- removed joint gripper_side_joint
- removed joint robotiq_85_base_joint
- removed joint robotiq_85_left_finger_joint
- removed joint robotiq_85_left_finger_tip_joint
- removed joint robotiq_85_left_inner_knuckle_joint
- removed joint robotiq_85_left_knuckle_joint
- removed joint robotiq_85_right_finger_joint
- removed joint robotiq_85_right_finger_tip_joint
- removed joint robotiq_85_right_inner_knuckle_joint
- removed joint robotiq_85_right_knuckle_joint
- removed joint ur_to_robotiq_joint
- joint shoulder_pan_joint: origin xyz=0 0 0.1625 rpy=0 0 0 -> xyz=0 0 0.089159 rpy=0 0 0
- joint wrist_1_joint: origin xyz=-0.3922 0 0.1333 rpy=0 0 0 -> xyz=-0.39225 0 0.10915 rpy=0 0 0
- joint wrist_2_joint: origin xyz=0 -0.0997 -2.044881182297852e-11 rpy=1.570796327 0 0 -> xyz=0 -0.09465 -1.941303950897609e-11 rpy=1.570796327 0 0
- joint wrist_3_joint: origin xyz=0 0.0996 -2.042830148012698e-11 rpy=1.570796326589793 3.141592653589793 3.141592653589793 -> xyz=0 0.0823 -1.688001216681175e-11 rpy=1.570796326589793 3.141592653589793 3.141592653589793

File: urdf/asbr.urdf.xacro (robot description, xacro)
@@ -1,130 +1,11 @@
 <?xml version="1.0"?>
 <robot name="ur5e_robot" xmlns:xacro="http://www.ros.org/wiki/xacro">
-    <xacro:arg name="name" default="ur5e_robot"/>
-    <!-- Include the URDF for the UR robot -->
-    <xacro:include filename="$(find ur_description)/urdf/ur_macro.xacro"/>
-    <!-- Defining Main parameters -->
-    <xacro:arg name="ur_type" default="ur5"/>
-    <xacro:arg name="tf_prefix" default=""/>
-    <xacro:arg name="joint_limit_params" default="$(find ur_description)/config/$(arg ur_type)/joint_limits.yaml"/>
-    <xacro:arg name="kinematics_params" default="$(find ur_description)/config/$(arg ur_type)/default_kinematics.yaml"/>
-    <xacro:arg name="physical_params" default="$(find ur_description)/config/$(arg ur_type)/physical_parameters.yaml"/>
-    <xacro:arg name="visual_params" default="$(find ur_description)/config/$(arg ur_type)/visual_parameters.yaml"/>
-    <xacro:arg name="transmission_hw_interface" default="hardware_interface/PositionJointInterface"/>
-    <xacro:arg name="safety_limits" default="true"/> <!-- I set this to true cause it makes sense to do so -->
-    <xacro:arg name="safety_pos_margin" default="0.15"/>
-    <xacro:arg name="safety_k_position" default="20"/>
-    <!-- Simulation and Control Parameters -->
-    <xacro:arg name="use_fake_hardware" default="false"/> <!-- Using the real UR5 or UR5e-->
-    <xacro:arg name="fake_sensor_commands" default="false"/>
-    <xacro:arg name="sim_gazebo" default="false"/>
-    <xacro:arg name="sim_ignition" default="false"/>
-    <xacro:arg name="sim_isaac" default="false"/>
-    <xacro:arg name="headless_mode" default="true"/> <!-- Setting the headless mode to true for real robot-->
-    <xacro:arg name="robot_ip" default="172.22.22.2"/> <!-- Current robot_ip on the UR5-->
-    <xacro:arg name="script_filename" default=""/>
-    <xacro:arg name="output_recipe_filename" default=""/>
-    <xacro:arg name="input_recipe_filename" default=""/>
-    <xacro:arg name="reverse_ip" default="172.22.22.10"/> <!-- I think this is the other ip ad which is for my laptop 172.22.22.10-->
-    <xacro:arg name="script_command_port" default="50004"/>
-    <xacro:arg name="reverse_port" default="50001"/>
-    <xacro:arg name="script_sender_port" default="50002"/>
-    <xacro:arg name="trajectory_port" default="50003"/>
-    <!-- Tool Communication Related Parameters-->
-    <xacro:arg name="use_tool_communication" default="false"/>
-    <xacro:arg name="tool_voltage" default="0"/>
-    <xacro:arg name="tool_parity" default="0"/>
-    <xacro:arg name="tool_baud_rate" default="115200"/>
-    <xacro:arg name="tool_stop_bits" default="1"/>
-    <xacro:arg name="tool_rx_idle_chars" default="1.5"/>
-    <xacro:arg name="tool_tx_idle_chars" default="3.5"/>
-    <xacro:arg name="tool_device_name" default="/tmp/ttyUR"/>
-    <xacro:arg name="tool_tcp_port" default="54321"/>
-    <xacro:arg name="com_port" default="/dev/ttyUSB0"/> <!-- Change this based on what your ports say (lsusb)-->
-    <xacro:arg name="include_ros2_control" default="true"/>
-    <xacro:arg name="initial_positions_file" default="$(find ur_description)/config/initial_positions.yaml"/>
-    <xacro:property name="initial_positions_file" default="$(arg initial_positions_file)"/>
-    <!-- Create link fixed to the world -->
-    <link name="world" />
-    <!-- Instantiate the UR robot macro -->
-    <xacro:ur_robot
-        name="$(arg name)"
-        tf_prefix="$(arg tf_prefix)"
-        parent="world"
-        joint_limits_parameters_file="$(arg joint_limit_params)"
-        kinematics_parameters_file="$(arg kinematics_params)"
-        physical_parameters_file="$(arg physical_params)"
-        visual_parameters_file="$(arg visual_params)"
-        transmission_hw_interface="$(arg transmission_hw_interface)"
-        safety_limits="$(arg safety_limits)"
-        safety_pos_margin="$(arg safety_pos_margin)"
-        safety_k_position="$(arg safety_k_position)"
-        use_fake_hardware="$(arg use_fake_hardware)"
-        fake_sensor_commands="$(arg fake_sensor_commands)"
-        sim_gazebo="$(arg sim_gazebo)"
-        sim_ignition="$(arg sim_ignition)"
-        headless_mode="$(arg headless_mode)"
-        initial_positions="${xacro.load_yaml(initial_positions_file)}"
-        use_tool_communication="$(arg use_tool_communication)"
-        tool_voltage="$(arg tool_voltage)"
-        tool_parity="$(arg tool_parity)"
-        tool_baud_rate="$(arg tool_baud_rate)"
-        tool_stop_bits="$(arg tool_stop_bits)"
-        tool_rx_idle_chars="$(arg tool_rx_idle_chars)"
-        tool_tx_idle_chars="$(arg tool_tx_idle_chars)"
-        tool_device_name="$(arg tool_device_name)"
-        tool_tcp_port="$(arg tool_tcp_port)"
-        robot_ip="$(arg robot_ip)"
-        script_filename="$(arg script_filename)"
-        output_recipe_filename="$(arg output_recipe_filename)"
-        input_recipe_filename="$(arg input_recipe_filename)"
-        reverse_ip="$(arg reverse_ip)"
-        script_command_port="$(arg script_command_port)"
-        reverse_port="$(arg reverse_port)"
-        script_sender_port="$(arg script_sender_port)"
-        trajectory_port="$(arg trajectory_port)">
-        <origin xyz="0 0 0" rpy="0 0 0"/>
-    </xacro:ur_robot>
-    Including the description for the gripper and adapter macro
-    <xacro:include filename="$(find robotiq_description)/urdf/robotiq_2f_85_macro.urdf.xacro"/>
-    <xacro:include filename="$(find robotiq_description)/urdf/ur_to_robotiq_adapter.urdf.xacro"/>
-    <!-- Instantiating the gripper macro and the adapter macro-->
-    <xacro:ur_to_robotiq prefix="" connected_to="tool0"/> <!-- This is the adapter-->
-    <!-- Attach the ur_to_robotiq_link (last link in the adapter urdf) to the gripper urdf-->
-    <xacro:robotiq_gripper
-        name="ur5e_gripper"
-        prefix=""
-        parent="gripper_mount_link"
-        sim_ignition="$(arg sim_ignition)"
-        sim_isaac="$(arg sim_isaac)"
-        use_fake_hardware="$(arg use_fake_hardware)"
-        fake_sensor_commands="$(arg fake_sensor_commands)"
-        com_port="$(arg com_port)"
-        >
-        <origin xyz="0 0 0" rpy="0 0 0"/>
-    </xacro:robotiq_gripper>
+    <!-- Include the arm (UR5 or UR5e -->
+     <xacro:include filename="arm.urdf.xacro"/>
+    <!-- Adding the gripper + adapter-->
+    <xacro:include filename="gripper.urdf.xacro"/>
     <!-- Adding the camera -->
     <xacro:include filename="camera.xacro"/>
     <!-- *************Gazebo classic and Ignition gazebo if ever needed*********** -->
-    <xacro:if value="$(arg sim_gazebo)">
-        <!-- Gazebo plugins -->
-        <gazebo reference="world">
-        </gazebo>
-        <gazebo>
-            <plugin filename="libgazebo_ros2_control.so" name="gazebo_ros2_control">
-                <parameters>$(arg simulation_controllers)</parameters>
-            </plugin>
-        </gazebo>
-    </xacro:if>
-    <xacro:if value="$(arg sim_ignition)">
-        <!-- Gazebo plugins -->
-        <gazebo reference="world">
-        </gazebo>
-        <gazebo>
-            <plugin filename="libign_ros2_control-system.so" name="ign_ros2_control::IgnitionROS2ControlPlugin">
-                <parameters>$(arg simulation_controllers)</parameters>
-                <controller_manager_node_name>$(arg tf_prefix)controller_manager</controller_manager_node_name>
-            </plugin>
-        </gazebo>
-    </xacro:if>
+    <xacro:include filename="gazebo.xacro"/>
 </robot>

Commit message: urdf updated

File: urdf/asbr.urdf (robot description, URDF)
Before this commit: robot ur5e_robot, 25 links, 24 joints
Links:
- added link gripper_mount_link
- added link robotiq_85_base_link, mass 6.6320197e-01; collision mesh filename=file:///opt/ros/humble/share/robotiq_description/meshes/col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; visual mesh filename=file:///opt/ros/humble/share/robotiq_description/meshes/vis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
- added link robotiq_85_left_finger_link, mass 4.260376752e-02; collision mesh filename=file:///opt/ros/humble/share/robotiq_description/meshes/col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; visual mesh filename=file:///opt/ros/humble/share/robotiq_description/meshes/vis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
- added link robotiq_85_left_finger_tip_link, mass 4.268588744e-02; collision mesh filename=file:///opt/ros/humble/share/robotiq_description/meshes/col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; visual mesh filename=file:///opt/ros/humble/share/robotiq_description/meshes/vis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
- added link robotiq_85_left_inner_knuckle_link, mass 2.969376448e-02; collision mesh filename=file:///opt/ros/humble/share/robotiq_description/meshes/col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; visual mesh filename=file:///opt/ros/humble/share/robotiq_description/meshes/vis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
- added link robotiq_85_left_knuckle_link, mass 1.384773208e-02; collision mesh filename=file:///opt/ros/humble/share/robotiq_description/meshes/col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; visual mesh filename=file:///opt/ros/humble/share/robotiq_description/meshes/vis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
- added link robotiq_85_right_finger_link, mass 4.260376752000000e-02; collision mesh filename=file:///opt/ros/humble/share/robotiq_description/meshes/col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; visual mesh filename=file:///opt/ros/humble/share/robotiq_description/meshes/vis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
- added link robotiq_85_right_finger_tip_link, mass 4.268588744e-02; collision mesh filename=file:///opt/ros/humble/share/robotiq_description/meshes/col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; visual mesh filename=file:///opt/ros/humble/share/robotiq_description/meshes/vis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
- added link robotiq_85_right_inner_knuckle_link, mass 2.969376448e-02; collision mesh filename=file:///opt/ros/humble/share/robotiq_description/meshes/col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; visual mesh filename=file:///opt/ros/humble/share/robotiq_description/meshes/vis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
- added link robotiq_85_right_knuckle_link, mass 1.384773208e-02; collision mesh filename=file:///opt/ros/humble/share/robotiq_description/meshes/col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; visual mesh filename=file:///opt/ros/humble/share/robotiq_description/meshes/vis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
- added link ur_to_robotiq_link, mass 0.01; collision mesh filename=package://robotiq_description/meshes/collision/ur_to_roboti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; visual mesh filename=package://robotiq_description/meshes/visual/ur_to_robotiq_a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
Joints:
- added joint gripper_side_joint: type fixed, parent ur_to_robotiq_link, child gripper_mount_link, origin xyz=0 0 0.011 rpy=0 0 0
- added joint robotiq_85_base_joint: type fixed, parent gripper_mount_link, child robotiq_85_base_link, origin xyz=0 0 0 rpy=0 0 0
- added joint robotiq_85_left_finger_joint: type fixed, parent robotiq_85_left_knuckle_link, child robotiq_85_left_finger_link, origin xyz=0.03152616 0.0 -0.00376347 rpy=0 0 0
- added joint robotiq_85_left_finger_tip_joint: type continuous, parent robotiq_85_left_finger_link, child robotiq_85_left_finger_tip_link, origin xyz=0.00563134 0.0 0.04718515 rpy=0 0 0, axis 0 -1 0, mimic joint=robotiq_85_left_knuckle_joint multiplier=-1
- added joint robotiq_85_left_inner_knuckle_joint: type continuous, parent robotiq_85_base_link, child robotiq_85_left_inner_knuckle_link, origin xyz=0.0127 0.0 0.06142 rpy=0 0 0, axis 0 -1 0, mimic joint=robotiq_85_left_knuckle_joint
- added joint robotiq_85_left_knuckle_joint: type revolute, parent robotiq_85_base_link, child robotiq_85_left_knuckle_link, origin xyz=0.03060114 0.0 0.05490452 rpy=0 0 0, axis 0 -1 0, limit lower=0.0 upper=0.8 effort=50 velocity=0.5
- added joint robotiq_85_right_finger_joint: type fixed, parent robotiq_85_right_knuckle_link, child robotiq_85_right_finger_link, origin xyz=-0.03152616 0.0 -0.00376347 rpy=0 0 0
- added joint robotiq_85_right_finger_tip_joint: type continuous, parent robotiq_85_right_finger_link, child robotiq_85_right_finger_tip_link, origin xyz=-0.00563134 0.0 0.04718515 rpy=0 0 0, axis 0 -1 0, mimic joint=robotiq_85_left_knuckle_joint
- added joint robotiq_85_right_inner_knuckle_joint: type continuous, parent robotiq_85_base_link, child robotiq_85_right_inner_knuckle_link, origin xyz=-0.0127 0.0 0.06142 rpy=0 0 0, axis 0 -1 0, mimic joint=robotiq_85_left_knuckle_joint multiplier=-1
- added joint robotiq_85_right_knuckle_joint: type revolute, parent robotiq_85_base_link, child robotiq_85_right_knuckle_link, origin xyz=-0.03060114 0.0 0.05490452 rpy=0 0 0, axis 0 -1 0, limit lower=-0.8 upper=0.0 effort=50 velocity=0.5, mimic joint=robotiq_85_left_knuckle_joint multiplier=-1
- added joint ur_to_robotiq_joint: type fixed, parent tool0, child ur_to_robotiq_link, origin xyz=0 0 0 rpy=0 0 0.0

Commit message: update gripper

File: urdf/asbr.urdf (robot description, URDF)
Before this commit: robot ur5e_robot, 36 links, 35 joints
Links:
- link robotiq_85_base_link: geometry collision mesh filename=file:///home/r9/asbr_ws/install/robotiq_description/share/r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; visual mesh filename=file:///home/r9/asbr_ws/install/robotiq_description/share/r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
- link robotiq_85_left_finger_link: geometry collision mesh filename=file:///home/r9/asbr_ws/install/robotiq_description/share/r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; visual mesh filename=file:///home/r9/asbr_ws/install/robotiq_description/share/r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
- link robotiq_85_left_finger_tip_link: geometry collision mesh filename=file:///home/r9/asbr_ws/install/robotiq_description/share/r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; visual mesh filename=file:///home/r9/asbr_ws/install/robotiq_description/share/r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
- link robotiq_85_left_inner_knuckle_link: geometry collision mesh filename=file:///home/r9/asbr_ws/install/robotiq_description/share/r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; visual mesh filename=file:///home/r9/asbr_ws/install/robotiq_description/share/r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
- link robotiq_85_left_knuckle_link: geometry collision mesh filename=file:///home/r9/asbr_ws/install/robotiq_description/share/r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; visual mesh filename=file:///home/r9/asbr_ws/install/robotiq_description/share/r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
- link robotiq_85_right_finger_link: geometry collision mesh filename=file:///home/r9/asbr_ws/install/robotiq_description/share/r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; visual mesh filename=file:///home/r9/asbr_ws/install/robotiq_description/share/r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
- link robotiq_85_right_finger_tip_link: geometry collision mesh filename=file:///home/r9/asbr_ws/install/robotiq_description/share/r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; visual mesh filename=file:///home/r9/asbr_ws/install/robotiq_description/share/r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
- link robotiq_85_right_inner_knuckle_link: geometry collision mesh filename=file:///home/r9/asbr_ws/install/robotiq_description/share/r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; visual mesh filename=file:///home/r9/asbr_ws/install/robotiq_description/share/r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
- link robotiq_85_right_knuckle_link: geometry collision mesh filename=file:///home/r9/asbr_ws/install/robotiq_description/share/r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; visual mesh filename=file:///home/r9/asbr_ws/install/robotiq_description/share/r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
- link ur_to_robotiq_link: geometry collision mesh filename=package://robotiq_description/meshes/collision/2f_85/ur_to_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; visual mesh filename=package://robotiq_description/meshes/visual/2f_85/ur_to_rob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

File: urdf/gripper.urdf.xacro (robot description, xacro)
@@ -2,6 +2,6 @@
 <robot xmlns:xacro="http://www.ros.org/wiki/xacro" name="robotiq_gripper">
     <!-- Include the macro definitions -->
-    <xacro:include filename="$(find robotiq_description)/urdf/robotiq_2f_85_macro.urdf.xacro"/>
-    <xacro:include filename="$(find robotiq_description)/urdf/ur_to_robotiq_adapter.urdf.xacro"/>
+    <xacro:include filename="/home/r9/asbr_ws/src/robotiq_ws/src/robotiq_description/urdf/robotiq_2f_85_macro.urdf.xacro"/>
+    <xacro:include filename="/home/r9/asbr_ws/src/robotiq_ws/src/robotiq_description/urdf/ur_to_robotiq_adapter.urdf.xacro"/>
     <!-- Instantiating the adapter macro-->
     <xacro:ur_to_robotiq prefix="" parent="tool0" child="gripper_mount_link" rotation="0.0"/> <!-- This is the adapter -->
@@ -14,7 +14,6 @@
         sim_isaac="$(arg sim_isaac)"
         use_fake_hardware="$(arg use_fake_hardware)"
-        fake_sensor_commands="$(arg fake_sensor_commands)"
         com_port="$(arg com_port)"
-    >
+        >
         <origin xyz="0 0 0" rpy="0 0 0"/>
     </xacro:robotiq_gripper>
