Commit message: assignment 1 update

File: urdf/arm.urdf.xacro (robot description, xacro)
@@ -1,9 +1,9 @@
 <?xml version="1.0"?>
 <robot name="ur5e_robot" xmlns:xacro="http://www.ros.org/wiki/xacro">
-    <xacro:arg name="name" default="ur5e_robot"/>
+    <xacro:arg name="name" default="asbr"/>
     <!-- Include the URDF for the UR robot -->
     <xacro:include filename="$(find ur_description)/urdf/ur_macro.xacro"/>
     <!-- Defining Main parameters -->
-    <xacro:arg name="ur_type" default="ur5"/>
+    <xacro:arg name="ur_type" default="ur5e"/>
     <xacro:arg name="tf_prefix" default=""/>
     <xacro:arg name="joint_limit_params" default="$(find ur_description)/config/$(arg ur_type)/joint_limits.yaml"/>
@@ -19,5 +19,5 @@
     <xacro:arg name="fake_sensor_commands" default="false"/>
     <xacro:arg name="sim_gazebo" default="false"/>
-    <xacro:arg name="sim_ignition" default="false"/>
+    <xacro:arg name="sim_ignition" default="true"/>
     <xacro:arg name="sim_isaac" default="false"/>
     <xacro:arg name="headless_mode" default="true"/> <!-- Setting the headless mode to true for real robot-->

File: urdf/asbr.urdf.xacro (robot description, xacro)
@@ -1,11 +1,178 @@
 <?xml version="1.0"?>
-<robot name="ur5e_robot" xmlns:xacro="http://www.ros.org/wiki/xacro">
-    <!-- Include the arm (UR5 or UR5e -->
-     <xacro:include filename="arm.urdf.xacro"/>
-    <!-- Adding the gripper + adapter-->
-    <xacro:include filename="gripper.urdf.xacro"/>
-    <!-- Adding the camera -->
-    <xacro:include filename="camera.xacro"/>
-    <!-- *************Gazebo classic and Ignition gazebo if ever needed*********** -->
-    <xacro:include filename="gazebo.xacro"/>
+<robot name="asbr" xmlns:xacro="http://www.ros.org/wiki/xacro">
+  <!-- robot name parameter -->
+  <xacro:arg name="name" default="asbr"/>
+  <!-- import main macro -->
+  <xacro:include filename="$(find ur_description)/urdf/ur_macro.xacro"/>
+  <!-- possible 'ur_type' values: ur3, ur3e, ur5, ur5e, ur10, ur10e, ur16e, ur20, ur30 -->
+  <!-- the default value should raise an error in case this was called without defining the type -->
+  <xacro:arg name="ur_type" default="ur5e"/>
+  <!-- parameters -->
+  <xacro:arg name="tf_prefix" default="" />
+  <xacro:arg name="joint_limit_params" default="$(find ur_description)/config/$(arg ur_type)/joint_limits.yaml"/>
+  <xacro:arg name="kinematics_params" default="$(find ur_description)/config/$(arg ur_type)/default_kinematics.yaml"/>
+  <xacro:arg name="physical_params" default="$(find ur_description)/config/$(arg ur_type)/physical_parameters.yaml"/>
+  <xacro:arg name="visual_params" default="$(find ur_description)/config/$(arg ur_type)/visual_parameters.yaml"/>
+  <xacro:arg name="transmission_hw_interface" default=""/>
+  <xacro:arg name="safety_limits" default="false"/>
+  <xacro:arg name="safety_pos_margin" default="0.15"/>
+  <xacro:arg name="safety_k_position" default="20"/>
+  <!-- ros2_control related parameters -->
+  <xacro:arg name="headless_mode" default="false" />
+  <xacro:arg name="robot_ip" default="0.0.0.0" />
+  <xacro:arg name="script_filename" default=""/>
+  <xacro:arg name="output_recipe_filename" default=""/>
+  <xacro:arg name="input_recipe_filename" default=""/>
+  <xacro:arg name="reverse_ip" default="0.0.0.0"/>
+  <xacro:arg name="script_command_port" default="50004"/>
+  <xacro:arg name="reverse_port" default="50001"/>
+  <xacro:arg name="script_sender_port" default="50002"/>
+  <xacro:arg name="trajectory_port" default="50003"/>
+  <!--   tool communication related parameters-->
+  <xacro:arg name="use_tool_communication" default="false" />
+  <xacro:arg name="tool_voltage" default="0" />
+  <xacro:arg name="tool_parity" default="0" />
+  <xacro:arg name="tool_baud_rate" default="115200" />
+  <xacro:arg name="tool_stop_bits" default="1" />
+  <xacro:arg name="tool_rx_idle_chars" default="1.5" />
+  <xacro:arg name="tool_tx_idle_chars" default="3.5" />
+  <xacro:arg name="tool_device_name" default="/tmp/ttyUR" />
+  <xacro:arg name="tool_tcp_port" default="54321" />
+  <!-- Simulation parameters -->
+  <xacro:arg name="use_fake_hardware" default="false" />
+  <xacro:arg name="fake_sensor_commands" default="false" />
+  <xacro:arg name="sim_gazebo" default="false" />
+  <xacro:arg name="sim_ignition" default="false" />
+  <xacro:arg name="simulation_controllers" default="" />
+  <!-- initial position for simulations (Fake Hardware, Gazebo, Ignition) -->
+  <xacro:arg name="initial_positions_file" default="$(find ur_description)/config/initial_positions.yaml"/>
+  <xacro:arg name="com_port" default="/dev/ttyUSB0"/> <!-- Change this based on what your ports say (lsusb)-->
+  <!-- convert to property to use substitution in function -->
+  <xacro:property name="initial_positions_file" default="$(arg initial_positions_file)"/>
+  <!-- Create link fixed to the world -->
+  <link name="world" />
+  <!-- Instantiate the UR robot macro -->
+  <xacro:ur_robot
+      name="$(arg name)"
+      tf_prefix="$(arg tf_prefix)"
+      parent="world"
+      joint_limits_parameters_file="$(arg joint_limit_params)"
+      kinematics_parameters_file="$(arg kinematics_params)"
+      physical_parameters_file="$(arg physical_params)"
+      visual_parameters_file="$(arg visual_params)"
+      transmission_hw_interface="$(arg transmission_hw_interface)"
+      safety_limits="$(arg safety_limits)"
+      safety_pos_margin="$(arg safety_pos_margin)"
+      safety_k_position="$(arg safety_k_position)"
+      use_fake_hardware="$(arg use_fake_hardware)"
+      fake_sensor_commands="$(arg fake_sensor_commands)"
+      sim_gazebo="$(arg sim_gazebo)"
+      sim_ignition="$(arg sim_ignition)"
+      headless_mode="$(arg headless_mode)"
+      initial_positions="${xacro.load_yaml(initial_positions_file)}"
+      use_tool_communication="$(arg use_tool_communication)"
+      tool_voltage="$(arg tool_voltage)"
+      tool_parity="$(arg tool_parity)"
+      tool_baud_rate="$(arg tool_baud_rate)"
+      tool_stop_bits="$(arg tool_stop_bits)"
+      tool_rx_idle_chars="$(arg tool_rx_idle_chars)"
+      tool_tx_idle_chars="$(arg tool_tx_idle_chars)"
+      tool_device_name="$(arg tool_device_name)"
+      tool_tcp_port="$(arg tool_tcp_port)"
+      robot_ip="$(arg robot_ip)"
+      script_filename="$(arg script_filename)"
+      output_recipe_filename="$(arg output_recipe_filename)"
+      input_recipe_filename="$(arg input_recipe_filename)"
+      reverse_ip="$(arg reverse_ip)"
+      script_command_port="$(arg script_command_port)"
+      reverse_port="$(arg reverse_port)"
+      script_sender_port="$(arg script_sender_port)"
+      trajectory_port="$(arg trajectory_port)">
+    <origin xyz="0 0 0" rpy="0 0 0"/>
+  </xacro:ur_robot>
+  <!-- Include the macro definitions -->
+  <xacro:include filename="$(find robotiq_description)/urdf/robotiq_2f_85_macro.urdf.xacro"/>
+  <xacro:include filename="$(find robotiq_description)/urdf/ur_to_robotiq_adapter.urdf.xacro"/>
+  <xacro:ur_to_robotiq prefix="" connected_to="tool0" rotation="0.0"/>
+  <!-- Instantiating the gripper macro-->
+  <xacro:robotiq_gripper
+      name="gripper"
+      prefix="robotiq"
+      parent="gripper_mount_link"
+      sim_ignition="true"
+      sim_isaac="false"
+      use_fake_hardware="$(arg use_fake_hardware)"
+      com_port="$(arg com_port)"
+      >
+    <origin xyz="0 0 0" rpy="0 0 0"/>
+  </xacro:robotiq_gripper>
+  <!-- Adding the intermediate link between the end effector and the sensor for potentially installing camera adapters -->
+  <link name="camera_link">
+  </link>
+  <joint name="camera_joint" type="fixed">
+    <axis xyz="0 0 1"/>
+    <origin xyz="-0.15 -0.05 0.015" rpy="0 0 0"/>
+    <parent link="tool0"/>
+    <child link="camera_link"/>
+  </joint>
+  <!-- Including the description for the realsense2 camera -->
+  <xacro:include filename="$(find realsense2_description)/urdf/_d435.urdf.xacro" />
+  <!-- Connecting the camera sensor to the camera link -->
+  <xacro:sensor_d435 parent="tool0" name="d435" use_nominal_extrinsics="true" add_plug="true" use_mesh="true">
+    <origin xyz="0.0 -0.06 0.0" rpy="-1.5708 -1.5708 0"/>
+  </xacro:sensor_d435>
+  <gazebo reference="camera_link">
+    <material>Gazebo/Red</material>
+    <sensor type="camera" name="camera">
+      <update_rate> 30.0 </update_rate>
+      <topic> image_raw </topic>
+      <pose> 0 0 0   0 -1.5708 1.5708 </pose>
+      <camera name="head">
+        <image>
+          <width> 1920 </width>
+          <height> 1080 </height>
+          <format>R8G8B8</format>
+        </image>
+        <clip>
+          <near> 0.02 </near>
+          <far> 3 </far>
+        </clip>
+        <noise>
+          <mean> 0.0 </mean>
+          <stddev> 0.01 </stddev>
+        </noise>
+        <lens>
+          <type> gnomolical </type>
+          <intrinsics>
+            <fx>1663</fx>
+            <fy>1663</fy>
+            <cx>960</cx>
+            <cy>540</cy>
+            <s>0</s>
+          </intrinsics>
+          <projection>
+            <p_fx>1663</p_fx>
+            <p_fy>1663</p_fy>
+            <p_cx>960</p_cx>
+            <p_cy>540</p_cy>
+          </projection>
+        </lens>
+      </camera>
+      <plugin filename="ignition-gazebo-sensors-system"
+              name="ignition::gazebo::systems::Sensors">
+      </plugin>
+    </sensor>
+  </gazebo>
+  <!-- *************Gazebo classic and Ignition gazebo if ever needed*********** -->
+  <xacro:if value="$(arg sim_ignition)">
+    <!-- Gazebo plugins -->
+    <gazebo reference="world">
+    </gazebo>
+    <gazebo>
+      <plugin filename="libign_ros2_control-system.so" name="ign_ros2_control::IgnitionROS2ControlPlugin">
+        <parameters>$(arg simulation_controllers)</parameters>
+        <controller_manager_node_name>$(arg tf_prefix)controller_manager</controller_manager_node_name>
+      </plugin>
+    </gazebo>
+  </xacro:if>
 </robot>

File: urdf/gripper.urdf.xacro (robot description, xacro)
@@ -2,15 +2,15 @@
 <robot xmlns:xacro="http://www.ros.org/wiki/xacro" name="robotiq_gripper">
     <!-- Include the macro definitions -->
-    <xacro:include filename="/home/r9/asbr_ws/src/robotiq_ws/src/robotiq_description/urdf/robotiq_2f_85_macro.urdf.xacro"/>
-    <xacro:include filename="/home/r9/asbr_ws/src/robotiq_ws/src/robotiq_description/urdf/ur_to_robotiq_adapter.urdf.xacro"/>
+    <xacro:include filename="$(find robotiq_description)/urdf/robotiq_2f_85_macro.urdf.xacro"/>
+    <xacro:include filename="$(find robotiq_description)/urdf/ur_to_robotiq_adapter.urdf.xacro"/>
     <!-- Instantiating the adapter macro-->
-    <xacro:ur_to_robotiq prefix="" parent="tool0" child="gripper_mount_link" rotation="0.0"/> <!-- This is the adapter -->
+    <xacro:ur_to_robotiq prefix="" connected_to="tool0" rotation="0.0"/> <!-- This is the adapter -->
     <!-- Instantiating the gripper macro-->
     <xacro:robotiq_gripper
-        name="ur5e_gripper"
-        prefix=""
+        name="gripper"
+        prefix="robotiq"
         parent="gripper_mount_link"
-        sim_ignition="$(arg sim_ignition)"
-        sim_isaac="$(arg sim_isaac)"
+        sim_ignition="true"
+        sim_isaac="false"
         use_fake_hardware="$(arg use_fake_hardware)"
         com_port="$(arg com_port)"
