Commit message: stuff

File: urdf/asbr.urdf.xacro (robot description, xacro)
@@ -14,6 +14,29 @@
     <xacro:arg name="safety_pos_margin" default="0.15"/>
     <xacro:arg name="safety_k_position" default="20"/>
+    <xacro:arg name="use_fake_hardware" default="false"/>
+    <xacro:arg name="fake_sensor_commands" default="false"/>
     <xacro:arg name="sim_gazebo" default="false"/>
     <xacro:arg name="sim_ignition" default="false"/>
+    <xacro:arg name="headless_mode" default="false"/>
+    <xacro:arg name="robot_ip" default="0.0.0.0"/>
+    <xacro:arg name="script_filename" default=""/>
+    <xacro:arg name="output_recipe_filename" default=""/>
+    <xacro:arg name="input_recipe_filename" default=""/>
+    <xacro:arg name="reverse_ip" default="0.0.0.0"/>
+    <xacro:arg name="script_command_port" default="50004"/>
+    <xacro:arg name="reverse_port" default="50001"/>
+    <xacro:arg name="script_sender_port" default="50002"/>
+    <xacro:arg name="trajectory_port" default="50003"/>
+    <xacro:arg name="use_tool_communication" default="false"/>
+    <xacro:arg name="tool_voltage" default="0"/>
+    <xacro:arg name="tool_parity" default="0"/>
+    <xacro:arg name="tool_baud_rate" default="115200"/>
+    <xacro:arg name="tool_stop_bits" default="1"/>
+    <xacro:arg name="tool_rx_idle_chars" default="1.5"/>
+    <xacro:arg name="tool_tx_idle_chars" default="3.5"/>
+    <xacro:arg name="tool_device_name" default="/tmp/ttyUR"/>
+    <xacro:arg name="tool_tcp_port" default="54321"/>
+    <xacro:arg name="initial_positions_file" default="$(find ur_description)/config/initial_positions.yaml"/>
+    <xacro:arg name="simulation_controllers" default=""/>
     <!-- Include the URDF for the UR robot -->
     <xacro:include filename="$(find ur_description)/urdf/ur_macro.xacro"/>
@@ -31,6 +54,51 @@
         safety_pos_margin="$(arg safety_pos_margin)"
         safety_k_position="$(arg safety_k_position)"
+        use_fake_hardware="$(arg use_fake_hardware)"
+        fake_sensor_commands="$(arg fake_sensor_commands)"
         sim_gazebo="$(arg sim_gazebo)"
         sim_ignition="$(arg sim_ignition)"
-    />
+        headless_mode="$(arg headless_mode)"
+        initial_positions="${xacro.load_yaml(initial_positions_file)}"
+        use_tool_communication="$(arg use_tool_communication)"
+        tool_voltage="$(arg tool_voltage)"
+        tool_parity="$(arg tool_parity)"
+        tool_baud_rate="$(arg tool_baud_rate)"
+        tool_stop_bits="$(arg tool_stop_bits)"
+        tool_rx_idle_chars="$(arg tool_rx_idle_chars)"
+        tool_tx_idle_chars="$(arg tool_tx_idle_chars)"
+        tool_device_name="$(arg tool_device_name)"
+        tool_tcp_port="$(arg tool_tcp_port)"
+        robot_ip="$(arg robot_ip)"
+        script_filename="$(arg script_filename)"
+        output_recipe_filename="$(arg output_recipe_filename)"
+        input_recipe_filename="$(arg input_recipe_filename)"
+        reverse_ip="$(arg reverse_ip)"
+        script_command_port="$(arg script_command_port)"
+        reverse_port="$(arg reverse_port)"
+        script_sender_port="$(arg script_sender_port)"
+        trajectory_port="$(arg trajectory_port)"
+    >
+        <origin xyz="0 0 0" rpy="0 0 0"/>
+    </xacro:ur_robot>
+    <xacro:if value="$(arg sim_gazebo)">
+        <!-- Gazebo plugins -->
+        <gazebo reference="world">
+        </gazebo>
+        <gazebo>
+            <plugin filename="libgazebo_ros2_control.so" name="gazebo_ros2_control">
+                <parameters>$(arg simulation_controllers)</parameters>
+            </plugin>
+        </gazebo>
+    </xacro:if>
+    <xacro:if value="$(arg sim_ignition)">
+        <!-- Ignition plugins -->
+        <gazebo reference="world">
+        </gazebo>
+        <gazebo>
+            <plugin filename="libign_ros2_control-system.so" name="ign_ros2_control::IgnitionROS2ControlPlugin">
+                <parameters>$(arg simulation_controllers)</parameters>
+                <controller_manager_node_name>$(arg tf_prefix)controller_manager</controller_manager_node_name>
+            </plugin>
+        </gazebo>
+    </xacro:if>
 </robot>

Commit message: modified urdf

File: urdf/asbr.urdf.xacro (robot description, xacro)
@@ -37,5 +37,5 @@
     <xacro:arg name="tool_device_name" default="/tmp/ttyUR"/>
     <xacro:arg name="tool_tcp_port" default="54321"/>
-    <xacro:arg name="initial_positions_file" default="$(find ur_description)/config/initial_positions.yaml"/>
+    <xacro:property name="initial_positions_file" default="$(arg initial_positions_file)"/>
     <xacro:arg name="simulation_controllers" default=""/>
     <!-- Include the URDF for the UR robot -->

Commit message: new modification

File: urdf/asbr.urdf.xacro (robot description, xacro)
@@ -2,5 +2,5 @@
 <robot name="ur5e_robot" xmlns:xacro="http://www.ros.org/wiki/xacro">
     <!-- Developer: Seyi R. Afolayan -->
-    <!-- Arguments required by ur.urdf.xacro -->
+    <!-- Arguments for UR5e hardware setup -->
     <xacro:arg name="name" default="ur5e_robot"/>
     <xacro:arg name="ur_type" default="ur5e"/>
@@ -37,6 +37,12 @@
     <xacro:arg name="tool_device_name" default="/tmp/ttyUR"/>
     <xacro:arg name="tool_tcp_port" default="54321"/>
-    <xacro:property name="initial_positions_file" default="$(arg initial_positions_file)"/>
-    <xacro:arg name="simulation_controllers" default=""/>
+    <xacro:arg name="initial_positions" default="${xacro.dict(
+        shoulder_pan_joint=0.0,
+        shoulder_lift_joint=-1.57,
+        elbow_joint=1.57,
+        wrist_1_joint=0.0,
+        wrist_2_joint=-1.57,
+        wrist_3_joint=0.0
+    )}"/>
     <!-- Include the URDF for the UR robot -->
     <xacro:include filename="$(find ur_description)/urdf/ur_macro.xacro"/>
@@ -59,5 +65,5 @@
         sim_ignition="$(arg sim_ignition)"
         headless_mode="$(arg headless_mode)"
-        initial_positions="${xacro.load_yaml(initial_positions_file)}"
+        initial_positions="$(arg initial_positions)"
         use_tool_communication="$(arg use_tool_communication)"
         tool_voltage="$(arg tool_voltage)"
@@ -81,24 +87,3 @@
         <origin xyz="0 0 0" rpy="0 0 0"/>
     </xacro:ur_robot>
-    <xacro:if value="$(arg sim_gazebo)">
-        <!-- Gazebo plugins -->
-        <gazebo reference="world">
-        </gazebo>
-        <gazebo>
-            <plugin filename="libgazebo_ros2_control.so" name="gazebo_ros2_control">
-                <parameters>$(arg simulation_controllers)</parameters>
-            </plugin>
-        </gazebo>
-    </xacro:if>
-    <xacro:if value="$(arg sim_ignition)">
-        <!-- Ignition plugins -->
-        <gazebo reference="world">
-        </gazebo>
-        <gazebo>
-            <plugin filename="libign_ros2_control-system.so" name="ign_ros2_control::IgnitionROS2ControlPlugin">
-                <parameters>$(arg simulation_controllers)</parameters>
-                <controller_manager_node_name>$(arg tf_prefix)controller_manager</controller_manager_node_name>
-            </plugin>
-        </gazebo>
-    </xacro:if>
 </robot>

Commit message: working urdf

File: urdf/asbr.urdf.xacro (robot description, xacro)
@@ -1,13 +1,15 @@
 <?xml version="1.0"?>
 <robot name="ur5e_robot" xmlns:xacro="http://www.ros.org/wiki/xacro">
-    <!-- Developer: Seyi R. Afolayan -->
-    <!-- Arguments for UR5e hardware setup -->
     <xacro:arg name="name" default="ur5e_robot"/>
+    <!-- Include the URDF for the UR robot -->
+    <xacro:include filename="$(find ur_description)/urdf/ur_macro.xacro"/>
+    <!-- ur parameters -->
     <xacro:arg name="ur_type" default="ur5e"/>
     <xacro:arg name="tf_prefix" default=""/>
-    <xacro:arg name="joint_limit_params" default="$(find ur_description)/config/ur5e/joint_limits.yaml"/>
-    <xacro:arg name="kinematics_params" default="$(find ur_description)/config/ur5e/default_kinematics.yaml"/>
-    <xacro:arg name="physical_params" default="$(find ur_description)/config/ur5e/physical_parameters.yaml"/>
-    <xacro:arg name="visual_params" default="$(find ur_description)/config/ur5e/visual_parameters.yaml"/>
+    <xacro:arg name="tf_prefix" default="" />
+    <xacro:arg name="joint_limit_params" default="$(find ur_description)/config/$(arg ur_type)/joint_limits.yaml"/>
+    <xacro:arg name="kinematics_params" default="$(find ur_description)/config/$(arg ur_type)/default_kinematics.yaml"/>
+    <xacro:arg name="physical_params" default="$(find ur_description)/config/$(arg ur_type)/physical_parameters.yaml"/>
+    <xacro:arg name="visual_params" default="$(find ur_description)/config/$(arg ur_type)/visual_parameters.yaml"/>
     <xacro:arg name="transmission_hw_interface" default="hardware_interface/PositionJointInterface"/>
     <xacro:arg name="safety_limits" default="false"/>
@@ -37,7 +39,5 @@
     <xacro:arg name="tool_device_name" default="/tmp/ttyUR"/>
     <xacro:arg name="tool_tcp_port" default="54321"/>
-    <xacro:arg name="initial_positions" default="{shoulder_pan_joint: 0.0, shoulder_lift_joint: -1.57, elbow_joint: 1.57, wrist_1_joint: 0.0, wrist_2_joint: -1.57, wrist_3_joint: 0.0}"/>
-    <!-- Include the URDF for the UR robot -->
-    <xacro:include filename="$(find ur_description)/urdf/ur_macro.xacro"/>
+   <link name="world" />
     <!-- Instantiate the UR robot macro -->
     <xacro:ur_robot
@@ -58,5 +58,4 @@
         sim_ignition="$(arg sim_ignition)"
         headless_mode="$(arg headless_mode)"
-        initial_positions="$(arg initial_positions)"
         use_tool_communication="$(arg use_tool_communication)"
         tool_voltage="$(arg tool_voltage)"

Commit message: modified

File: urdf/asbr.urdf.xacro (robot description, xacro)
@@ -39,5 +39,10 @@
     <xacro:arg name="tool_device_name" default="/tmp/ttyUR"/>
     <xacro:arg name="tool_tcp_port" default="54321"/>
-   <link name="world" />
+    <!-- Include the URDF for the UR robot -->
+    <xacro:include filename="$(find ur_description)/urdf/ur_macro.xacro"/>
+    <!-- Load the initial_positions from the YAML file -->
+    <xacro:property name="initial_positions" value="$(load_yaml $(find ur_description)/config/initial_positions.yaml)"/>
+    <!-- create link fixed to the "world" -->
+    <link name="world" />
     <!-- Instantiate the UR robot macro -->
     <xacro:ur_robot
@@ -58,4 +63,5 @@
         sim_ignition="$(arg sim_ignition)"
         headless_mode="$(arg headless_mode)"
+        initial_positions="$(arg initial_positions)"
         use_tool_communication="$(arg use_tool_communication)"
         tool_voltage="$(arg tool_voltage)"
@@ -79,3 +85,24 @@
         <origin xyz="0 0 0" rpy="0 0 0"/>
     </xacro:ur_robot>
+    <xacro:if value="$(arg sim_gazebo)">
+        <!-- Gazebo plugins -->
+        <gazebo reference="world">
+        </gazebo>
+        <gazebo>
+            <plugin filename="libgazebo_ros2_control.so" name="gazebo_ros2_control">
+                <parameters>$(arg simulation_controllers)</parameters>
+            </plugin>
+        </gazebo>
+    </xacro:if>
+    <xacro:if value="$(arg sim_ignition)">
+        <!-- Gazebo plugins -->
+        <gazebo reference="world">
+        </gazebo>
+        <gazebo>
+            <plugin filename="libign_ros2_control-system.so" name="ign_ros2_control::IgnitionROS2ControlPlugin">
+                <parameters>$(arg simulation_controllers)</parameters>
+                <controller_manager_node_name>$(arg tf_prefix)controller_manager</controller_manager_node_name>
+            </plugin>
+        </gazebo>
+    </xacro:if>
 </robot>

Commit message: working urdf

File: urdf/asbr.urdf.xacro (robot description, xacro)
@@ -39,9 +39,6 @@
     <xacro:arg name="tool_device_name" default="/tmp/ttyUR"/>
     <xacro:arg name="tool_tcp_port" default="54321"/>
-    <!-- Include the URDF for the UR robot -->
-    <xacro:include filename="$(find ur_description)/urdf/ur_macro.xacro"/>
-    <!-- Load the initial_positions from the YAML file -->
-    <xacro:property name="initial_positions" value="$(load_yaml $(find ur_description)/config/initial_positions.yaml)"/>
-    <!-- create link fixed to the "world" -->
+    <xacro:property name="initial_positions_file" value="$(find ur_description)/config/initial_positions.yaml"/>
+    <xacro:property name="initial_positions" value="${xacro.load_yaml(initial_positions_file)}"/>
     <link name="world" />
     <!-- Instantiate the UR robot macro -->
@@ -63,5 +60,5 @@
         sim_ignition="$(arg sim_ignition)"
         headless_mode="$(arg headless_mode)"
-        initial_positions="$(arg initial_positions)"
+        initial_positions="${initial_positions}"
         use_tool_communication="$(arg use_tool_communication)"
         tool_voltage="$(arg tool_voltage)"

Commit message: Added the gripper

File: urdf/asbr.urdf.xacro (robot description, xacro)
@@ -16,5 +16,5 @@
     <xacro:arg name="safety_pos_margin" default="0.15"/>
     <xacro:arg name="safety_k_position" default="20"/>
-    <xacro:arg name="use_fake_hardware" default="false"/>
+    <xacro:arg name="use_fake_hardware" default="true"/> <!-- I changed this to true -->
     <xacro:arg name="fake_sensor_commands" default="false"/>
     <xacro:arg name="sim_gazebo" default="false"/>
@@ -82,4 +82,16 @@
         <origin xyz="0 0 0" rpy="0 0 0"/>
     </xacro:ur_robot>
+    <!-- Including the necessary modules for the complete ur5e absr_description -->
+    <xacro:include filename="$(find robotiq_description)/urdf/robotiq_2f_85_macro.urdf.xacro" />
+    <!-- Using the gripper macro-->
+    <xacro:robotiq_gripper name="ur5e_gripper" prefix="" parent="world" use_fake_hardware="$(arg use_fake_hardware">
+        <origin xyz="0 0 0" rpy="0 0 0"/>
+    </xacro:robotiq_gripper>
+    <!-- Connecting the end-effector to the gripper-->
+    <joint name="end_effector_gripper_joint" type="fixed">
+        <parent link="tool0"/>
+        <child link="ur5e_gripper"/>
+        <origin xyz="0 0 0" rpy="0 0 0"/>
+    </joint>
     <xacro:if value="$(arg sim_gazebo)">
         <!-- Gazebo plugins -->

Commit message: Added the adapter

File: urdf/asbr.urdf.xacro (robot description, xacro)
@@ -82,8 +82,14 @@
         <origin xyz="0 0 0" rpy="0 0 0"/>
     </xacro:ur_robot>
-    <!-- Including the necessary modules for the complete ur5e absr_description -->
+    <!-- Including the description for the gripper and adapter macro -->
     <xacro:include filename="$(find robotiq_description)/urdf/robotiq_2f_85_macro.urdf.xacro" />
-    <!-- Using the gripper macro-->
-    <xacro:robotiq_gripper name="ur5e_gripper" prefix="" parent="world" use_fake_hardware="$(arg use_fake_hardware">
+    <xacro:include filename="$(find robotiq_description)/urdf/ur_to_robotiq_adapter.urdf.xacro"/>
+    <!-- Instantiating the gripper macro and the adapter macro-->
+    <xacro:ur_to_robotiq prefix="" connected_to="tool0"/> <!-- This is the adapter-->
+    <xacro:robotiq_gripper
+        name="ur5e_gripper"
+        prefix=""
+        parent="ur_to_robotiq_link"
+        use_fake_hardware="$(arg use_fake_hardware)">
         <origin xyz="0 0 0" rpy="0 0 0"/>
     </xacro:robotiq_gripper>
@@ -91,5 +97,5 @@
     <joint name="end_effector_gripper_joint" type="fixed">
         <parent link="tool0"/>
-        <child link="ur5e_gripper"/>
+        <child link="robotiq_85_base_link"/>
         <origin xyz="0 0 0" rpy="0 0 0"/>
     </joint>

Commit message: remove the redundancy from the gripper stuff

File: urdf/asbr.urdf.xacro (robot description, xacro)
@@ -87,4 +87,5 @@
     <!-- Instantiating the gripper macro and the adapter macro-->
     <xacro:ur_to_robotiq prefix="" connected_to="tool0"/> <!-- This is the adapter-->
+    <!-- Attach the ur_to_robotiq_link (last link in the adapter urdf) to the gripper urdf-->
     <xacro:robotiq_gripper
         name="ur5e_gripper"
@@ -94,10 +95,4 @@
         <origin xyz="0 0 0" rpy="0 0 0"/>
     </xacro:robotiq_gripper>
-    <!-- Connecting the end-effector to the gripper-->
-    <joint name="end_effector_gripper_joint" type="fixed">
-        <parent link="tool0"/>
-        <child link="robotiq_85_base_link"/>
-        <origin xyz="0 0 0" rpy="0 0 0"/>
-    </joint>
     <xacro:if value="$(arg sim_gazebo)">
         <!-- Gazebo plugins -->

Commit message: Adding the camera urdf to main urdf

File: urdf/asbr.urdf.xacro (robot description, xacro)
@@ -105,4 +105,10 @@
         </gazebo>
     </xacro:if>
+    <!-- Including the description for the realsense2 camera -->
+    <xacro:include filename="$(find realsense2_description)/urdf/sensor_d435.urdf.xacro" />
+    <!-- Connecting the camera sensor to the camera link -->
+    <xacro:sensor_d435 parent="tool0" name="d435" use_nominal_extrinsics="true" add_plug="true" use_mesh="true">
+        <origin xyz="0.0 -0.06 0.0" rpy="-1.5708 -1.5708 0"/>
+    </xacro:sensor_d435>
     <xacro:if value="$(arg sim_ignition)">
         <!-- Gazebo plugins -->

Commit message: added the camera link to the urdf

File: urdf/asbr.urdf.xacro (robot description, xacro)
@@ -38,4 +38,5 @@
     <xacro:arg name="tool_device_name" default="/tmp/ttyUR"/>
     <xacro:arg name="tool_tcp_port" default="54321"/>
+    <!-- I am not sure if this is working at all -->
     <xacro:property name="initial_positions_file" value="$(find ur_description)/config/initial_positions.yaml"/>
     <xacro:property name="initial_positions" value="${xacro.load_yaml(initial_positions_file)}"/>
@@ -93,4 +94,20 @@
         <origin xyz="0 0 0" rpy="0 0 0"/>
     </xacro:robotiq_gripper>
+    <!-- Adding the intermediate link between the end effector and the sensor for potentially installing camera adapters -->
+    <link name="camera_link">
+    </link>
+    <joint name="camera_joint" type="fixed">
+        <axis xyz="0 0 1"/>
+        <origin xyz="-0.15 -0.05 0.015" rpy="0 0 0"/>
+        <parent link="tool0"/>
+        <child link="camera_link"/>
+    </joint>
+    <!-- Including the description for the realsense2 camera -->
+    <xacro:include filename="$(find realsense2_description)/urdf/_d435.urdf.xacro" />
+    <!-- Connecting the camera sensor to the camera link -->
+    <xacro:sensor_d435 parent="tool0" name="d435" use_nominal_extrinsics="true" add_plug="true" use_mesh="true">
+        <origin xyz="0.0 -0.06 0.0" rpy="-1.5708 -1.5708 0"/>
+    </xacro:sensor_d435>
+    <!-- *************Gazebo classic and Ignition gazebo if ever needed*********** -->
     <xacro:if value="$(arg sim_gazebo)">
         <!-- Gazebo plugins -->
@@ -103,10 +120,4 @@
         </gazebo>
     </xacro:if>
-    <!-- Including the description for the realsense2 camera -->
-    <xacro:include filename="$(find realsense2_description)/urdf/_d435.urdf.xacro" />
-    <!-- Connecting the camera sensor to the camera link -->
-    <xacro:sensor_d435 parent="tool0" name="d435" use_nominal_extrinsics="true" add_plug="true" use_mesh="true">
-        <origin xyz="0.0 -0.06 0.0" rpy="-1.5708 -1.5708 0"/>
-    </xacro:sensor_d435>
     <xacro:if value="$(arg sim_ignition)">
         <!-- Gazebo plugins -->

Commit message: organized the main xacro file

File: urdf/asbr.urdf.xacro (robot description, xacro)
@@ -40,6 +40,6 @@
     <xacro:arg name="tool_device_name" default="/tmp/ttyUR"/>
     <xacro:arg name="tool_tcp_port" default="54321"/>
-    <xacro:property name="initial_positions_file" value="$(find ur_description)/config/initial_positions.yaml"/>
-    <xacro:property name="initial_positions" value="${xacro.load_yaml(initial_positions_file)}"/>
+    <xacro:arg name="initial_positions_file" value="$(find ur_description)/config/initial_positions.yaml"/>
+    <xacro:property name="initial_positions_file" value="$(arg initial_positions_file)"/>
     <!-- Create link fixed to the world -->
     <link name="world" />
@@ -62,5 +62,5 @@
         sim_ignition="$(arg sim_ignition)"
         headless_mode="$(arg headless_mode)"
-        initial_positions="${initial_positions}"
+        initial_positions="${xacro.load_yaml(initial_positions_file)}"
         use_tool_communication="$(arg use_tool_communication)"
         tool_voltage="$(arg tool_voltage)"

Commit message: organized the main xacro file

File: urdf/asbr.urdf.xacro (robot description, xacro)
@@ -40,6 +40,6 @@
     <xacro:arg name="tool_device_name" default="/tmp/ttyUR"/>
     <xacro:arg name="tool_tcp_port" default="54321"/>
-    <xacro:arg name="initial_positions_file" value="$(find ur_description)/config/initial_positions.yaml"/>
-    <xacro:property name="initial_positions_file" value="$(arg initial_positions_file)"/>
+    <xacro:arg name="initial_positions_file" default="$(find ur_description)/config/initial_positions.yaml"/>
+    <xacro:property name="initial_positions_file" default="$(arg initial_positions_file)"/>
     <!-- Create link fixed to the world -->
     <link name="world" />

Commit message: asbtracted some code in the  main xacro

File: urdf/asbr.urdf.xacro (robot description, xacro)
@@ -96,19 +96,6 @@
         <origin xyz="0 0 0" rpy="0 0 0"/>
     </xacro:robotiq_gripper>
-    <!-- Adding the intermediate link between the end effector and the sensor for potentially installing camera adapters -->
-    <link name="camera_link">
-    </link>
-    <joint name="camera_joint" type="fixed">
-        <axis xyz="0 0 1"/>
-        <origin xyz="-0.15 -0.05 0.015" rpy="0 0 0"/>
-        <parent link="tool0"/>
-        <child link="camera_link"/>
-    </joint>
-    <!-- Including the description for the realsense2 camera -->
-    <xacro:include filename="$(find realsense2_description)/urdf/_d435.urdf.xacro" />
-    <!-- Connecting the camera sensor to the camera link -->
-    <xacro:sensor_d435 parent="tool0" name="d435" use_nominal_extrinsics="true" add_plug="true" use_mesh="true">
-        <origin xyz="0.0 -0.06 0.0" rpy="-1.5708 -1.5708 0"/>
-    </xacro:sensor_d435>
+    <!-- Adding the camera -->
+    <xacro:include filename="camera.xacro"/>
     <!-- *************Gazebo classic and Ignition gazebo if ever needed*********** -->
     <xacro:if value="$(arg sim_gazebo)">

File: urdf/camera.xacro (robot description, xacro)
@@ -1,4 +1,13 @@
 <?xml version="1.0"?>
 <robot xmlns:xacro="http://www.ros.org/wiki/xacro">
+    <!-- Adding the intermediate link between the end effector and the sensor for potentially installing camera adapters -->
+    <link name="camera_link">
+    </link>
+    <joint name="camera_joint" type="fixed">
+        <axis xyz="0 0 1"/>
+        <origin xyz="-0.15 -0.05 0.015" rpy="0 0 0"/>
+        <parent link="tool0"/>
+        <child link="camera_link"/>
+    </joint>
     <!-- Including the description for the realsense2 camera -->
     <xacro:include filename="$(find realsense2_description)/urdf/_d435.urdf.xacro" />
