Commit message: assignment camera fixes

File: urdf/asbr.urdf.xacro (robot description, xacro)
@@ -107,19 +107,20 @@
     <origin xyz="0 0 0" rpy="0 0 0"/>
   </xacro:robotiq_gripper>
-  <!-- Adding the intermediate link between the end effector and the sensor for potentially installing camera adapters -->
+  <!-- Including the description for the realsense2 camera -->
+  <xacro:include filename="$(find realsense2_description)/urdf/_d435.urdf.xacro" />
+  <!-- Connecting the camera sensor to the camera link -->
+  <xacro:sensor_d435 parent="tool0" name="d435" use_nominal_extrinsics="true" add_plug="true" use_mesh="true">
+    <origin xyz="0.0 -0.05 0.0" rpy="1.5708 -1.5708 0"/>
+  </xacro:sensor_d435>
+  <!-- Adding the intermediate link between the end effector and the sensor for potentially
+       installing camera adapters -->
   <link name="camera_link">
   </link>
   <joint name="camera_joint" type="fixed">
     <axis xyz="0 0 1"/>
-    <origin xyz="-0.15 -0.05 0.015" rpy="0 0 0"/>
-    <parent link="tool0"/>
+    <origin xyz="0 0 0" rpy="0 0 0"/>
+    <parent link="d435_color_optical_frame"/>
     <child link="camera_link"/>
   </joint>
-  <!-- Including the description for the realsense2 camera -->
-  <xacro:include filename="$(find realsense2_description)/urdf/_d435.urdf.xacro" />
-  <!-- Connecting the camera sensor to the camera link -->
-  <xacro:sensor_d435 parent="tool0" name="d435" use_nominal_extrinsics="true" add_plug="true" use_mesh="true">
-    <origin xyz="0.0 -0.06 0.0" rpy="-1.5708 -1.5708 0"/>
-  </xacro:sensor_d435>
   <gazebo reference="camera_link">
     <material>Gazebo/Red</material>
@@ -128,13 +129,14 @@
       <topic> image_raw </topic>
       <pose> 0 0 0   0 -1.5708 1.5708 </pose>
-      <camera name="head">
+      <camera name="camera">
+	<optical_frame_id> camera_link </optical_frame_id>
         <image>
-          <width> 1920 </width>
-          <height> 1080 </height>
+          <width> 1280 </width>
+          <height> 720 </height>
           <format>R8G8B8</format>
         </image>
         <clip>
           <near> 0.02 </near>
-          <far> 3 </far>
+          <far> 5 </far>
         </clip>
         <noise>
@@ -143,18 +145,12 @@
         </noise>
         <lens>
-          <type> gnomolical </type>
-          <intrinsics>
-            <fx>1663</fx>
-            <fy>1663</fy>
-            <cx>960</cx>
-            <cy>540</cy>
+	  <type> gnomolical </type>
+	  <intrinsics>
+            <fx>912.1078491210938</fx>
+            <fy>911.9324340820312</fy>
+            <cx>641.4862670898438</cx>
+            <cy>354.6959228515625</cy>
             <s>0</s>
-          </intrinsics>
-          <projection>
-            <p_fx>1663</p_fx>
-            <p_fy>1663</p_fy>
-            <p_cx>960</p_cx>
-            <p_cy>540</p_cy>
-          </projection>
+	  </intrinsics>
         </lens>
       </camera>

File: urdf/camera.xacro (robot description, xacro)
@@ -21,14 +21,14 @@
             <update_rate> 30.0 </update_rate>
             <topic> image_raw </topic>
-        <pose> 0 0 0   0 -1.5708 1.5708 </pose>
+            <pose> 0 0 0   0 -1.5708 1.5708 </pose>
             <camera name="head">
               <image>
-                <width> 1920 </width>
-                <height> 1080 </height>
+                <width> 1280 </width>
+                <height> 720 </height>
                 <format>R8G8B8</format>
               </image>
               <clip>
                 <near> 0.02 </near>
-                <far> 3 </far>
+                <far> 5 </far>
               </clip>
               <noise>
@@ -36,25 +36,19 @@
                 <stddev> 0.01 </stddev>
               </noise>
-          <lens>
-            <type> gnomolical </type>
-            <intrinsics>
-                  <fx>1663</fx>
-                  <fy>1663</fy>
-                  <cx>960</cx>
-                  <cy>540</cy>
+              <lens>
+		<type> gnomolical </type>
+		<intrinsics>
+                  <fx>912.1078491210938</fx>
+                  <fy>911.9324340820312</fy>
+                  <cx>641.4862670898438</cx>
+                  <cy>354.6959228515625</cy>
                   <s>0</s>
-            </intrinsics>
-            <projection>
-                  <p_fx>1663</p_fx>
-                  <p_fy>1663</p_fy>
-                  <p_cx>960</p_cx>
-                  <p_cy>540</p_cy>
-            </projection>
-          </lens>
+		</intrinsics>
+              </lens>
             </camera>
             <plugin filename="ignition-gazebo-sensors-system"
                     name="ignition::gazebo::systems::Sensors">
             </plugin>
-          </sensor>
+        </sensor>
     </gazebo>
 </robot>

Commit message: assingnment 3 mods

File: urdf/asbr.urdf.xacro (robot description, xacro)
@@ -46,5 +46,5 @@
   <xacro:arg name="simulation_controllers" default="" />
   <!-- initial position for simulations (Fake Hardware, Gazebo, Ignition) -->
-  <xacro:arg name="initial_positions_file" default="$(find ur_description)/config/initial_positions.yaml"/>
+  <xacro:arg name="initial_positions_file" default="$(find asbr_description)/config/initial_positions.yaml"/>
   <xacro:arg name="com_port" default="/dev/ttyUSB0"/> <!-- Change this based on what your ports say (lsusb)-->
   <!-- convert to property to use substitution in function -->
@@ -91,4 +91,11 @@
     <origin xyz="0 0 0" rpy="0 0 0"/>
   </xacro:ur_robot>
+  <link name="gripper_pick"/>
+  <joint name="gripper_pick_joint" type="fixed">
+    <axis xyz="0 0 1"/>
+    <origin xyz="0 0 0.175" rpy="0 -1.5707963267948970 0"/>
+    <parent link="wrist_3_link"/>
+    <child link="gripper_pick"/>
+  </joint>
   <!-- Include the macro definitions -->
   <xacro:include filename="$(find robotiq_description)/urdf/robotiq_2f_85_macro.urdf.xacro"/>

Commit message: sp 25

File: urdf/asbr.urdf.xacro (robot description, xacro)
@@ -94,5 +94,5 @@
   <joint name="gripper_pick_joint" type="fixed">
     <axis xyz="0 0 1"/>
-    <origin xyz="0 0 0.175" rpy="0 -1.5707963267948970 0"/>
+    <origin xyz="0 0 0.175" rpy="0 0 0"/>
     <parent link="wrist_3_link"/>
     <child link="gripper_pick"/>
